File: FS6-Adapter/FS6-Adapter.kicad_pcb (KiCad board)
At the start: 2 copper layers, 145.5 x 64 mm, 64 parts, among them J1 USB_C, J10 LEDs, J11 PWR_USB_PPM, J12 PPM_MODULE, J13 TRAINER, J14 I2C_STEMMA, J2 SWA, J3 SWB, J4 SWC, J5 SWD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

Commit message: Fix issues found
Parts:
- removed J12: PPM_MODULE, Connector_JST:JST_GH_BM04B-GHS-TBT_1x04-1MP_P1.25mm_Vertical
- added R20: 1K, Resistor_SMD:R_0603_1608Metric_Pad0.98x0.95mm_HandSolder, F.Cu at (125.6, 56.0)
- R10: value 100K -> 732K
- R8: value 20K -> 100K
- R9: value 100K -> 1M
- moved J14 31.8 mm to (95.0, 54.0)
- moved J2 31.3 mm to (167.8, 55.4), turned to 0 degrees
- moved D1 6.21 mm to (123.4, 100.4)
- moved D2 6.16 mm to (119.0, 101.4)
- moved SW5 5.00 mm to (73.0, 68.0)
- moved SW6 5.00 mm to (73.0, 78.0)
- moved J10 4.30 mm to (119.0, 61.2)
- moved C12 2.41 mm to (66.4, 57.8), turned to 0 degrees
- moved C11 1.80 mm to (70.2, 53.4)
- moved C13 1.70 mm to (71.2, 55.0)
- moved J3 1.60 mm to (192.2, 63.4)
- moved R19 1.60 mm to (71.2, 56.6)
- moved R10 0.80 mm to (74.6, 55.8)
- moved R9 0.80 mm to (74.6, 57.4)
- moved C9 0.60 mm to (63.0, 57.8)
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Connections:
- net 4IN1_LED renamed INT_PROTO_LED
- net ELRS_LED renamed INTMOD_LED
- net PPM_RX_LED renamed EXTMOD_LED
- J10 pad 4: PWR_EN -> Net-(J10-Pin_4)
- J11 pad 33: PPM_RX_5V -> unconnected-(J11-Pin_33-Pad33)
- J11 pad 34: PPM_RX_5V -> unconnected-(J11-Pin_34-Pad34)
- J11 pad 35: PPM_RX_5V -> unconnected-(J11-Pin_35-Pad35)
- J11 pad 36: PPM_RX_5V -> unconnected-(J11-Pin_36-Pad36)
- J6 pad 1: unconnected-(J6-Pin_1-Pad1) -> Net-(J6-Pin_1)
- J7 pad 1: unconnected-(J7-Pin_1-Pad1) -> Net-(J7-Pin_1)
- R11 pad 1: POTA_P -> Net-(J6-Pin_1)
- R13 pad 1: POTB_N -> Net-(J7-Pin_1)
Routing:
- net /SWA: track 103.1 -> 65.0 mm
- net SCL: track 143.0 -> 168.8 mm, vias 2 -> 4
- net SDA: track 143.0 -> 162.7 mm
- net Net-(J10-Pin_4): track 0.00 -> 16.1 mm, vias 0 -> 2
- net /USB and ADC/V_USB: track 66.9 -> 57.5 mm
- net INT_PROTO_LED: track 11.8 -> 7.48 mm
- net INTMOD_LED: track 12.1 -> 7.79 mm
- net EXTMOD_LED: track 11.7 -> 7.38 mm
- net CHARGING_LED: track 12.3 -> 8.00 mm
- net CHG_DONE_LED: track 12.0 -> 7.69 mm
- net /KEY_ENTER: track 52.9 -> 49.8 mm
- net VBUS: track 30.1 -> 33.1 mm
- net Net-(J7-Pin_1): track 0.00 -> 2.86 mm
- net Net-(J6-Pin_1): track 0.00 -> 2.80 mm
- net /KEY_EXIT: track 61.0 -> 58.6 mm
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- removed copper zone on F.Cu, net PPM_RX_5V
Other:
- outline, holes or cut-outs redrawn
