File: FS6-Adapter/FS6-Adapter.kicad_sch (KiCad schematic)
At the start: 27 parts, among them J10 LEDs, J11 PWR_USB_PPM, J12 PPM_MODULE, J13 TRAINER, J14 I2C_STEMMA, J2 SWA, J3 SWB, J4 SWC, J5 SWD, J6 VRA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

Commit message: Fix issues found
Parts:
- removed J12: PPM_MODULE, Connector_JST:JST_GH_BM04B-GHS-TBT_1x04-1MP_P1.25mm_Vertical, symbol Connector_Generic:Conn_01x04
- added R20: 1K, Resistor_SMD:R_0603_1608Metric_Pad0.98x0.95mm_HandSolder, symbol Device:R_US
Connections:
- net POTA_P: no longer R11.1
- net POTB_N: no longer R13.1
- net PWR_EN: now also R20.2; no longer J10.4 (Pin_4)
- net at J6.1 (Pin_1): now also R11.1
- net at J7.1 (Pin_1): now also R13.1
- net 4IN1_LED renamed INT_PROTO_LED
- net ELRS_LED renamed INTMOD_LED
- removed net PPM_RX_5V: J11.33 (Pin_33), J11.34 (Pin_34), J11.35 (Pin_35), J11.36 (Pin_36)
- net PPM_RX_LED renamed EXTMOD_LED
- new net: J10.4 (Pin_4), R20.1
