File: FS6-Adapter/usb_adc.kicad_sch (KiCad schematic)
At the start: 37 parts, among them J1 USB_C, Q1 MBT3904DW1, U1 CP2102N-Axx-xQFN24, U2 ADS1015IDGS, U3 ADS1015IDGS

Commit message: Fix issues found
Parts:
- R10: value 100K -> 732K
- R8: value 20K -> 100K
- R9: value 100K -> 1M
Changed lines of the file:
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@@
 		(dnp no)
 		(property "Reference" "R9"
-			(at 128.778 151.384 90)
-			(effects
-				(font
-					(size 1.27 1.27)
-				)
-			)
-		)
-		(property "Value" "100K"
+			(at 127 147.828 90)
+			(effects
+				(font
+					(size 1.27 1.27)
+				)
+			)
+		)
+		(property "Value" "1M"
 			(at 128.778 147.574 90)
 			(effects
@@
 		(dnp no)
 		(property "Reference" "R10"
-			(at 128.778 161.544 90)
-			(effects
-				(font
-					(size 1.27 1.27)
-				)
-			)
-		)
-		(property "Value" "100K"
+			(at 125.984 158.75 90)
+			(effects
+				(font
+					(size 1.27 1.27)
+				)
+			)
+		)
+		(property "Value" "732K"
 			(at 128.778 157.734 90)
 			(effects
@@
 		(dnp no)
 		(property "Reference" "R8"
-			(at 128.778 142.494 90)
-			(effects
-				(font
-					(size 1.27 1.27)
-				)
-			)
-		)
-		(property "Value" "20K"
+			(at 126.492 139.446 90)
+			(effects
+				(font
+					(size 1.27 1.27)
+				)
+			)
+		)
+		(property "Value" "100K"
 			(at 128.778 138.684 90)
 			(effects
