File: Muffin-Core/GPIO.kicad_sch (KiCad schematic)
At the start: 11 parts, among them J2 BUTTONS_AND_LEDS, J3 PWR_USB_PPM, SW1 PWR_SW_ON, SW2 ~{PWR_SW_DET}, U2 MCP23017_ML, U3 MCP23017_ML

Commit message: Fix issues found
Parts:
- added R14: 1K, Resistor_SMD:R_0603_1608Metric_Pad0.98x0.95mm_HandSolder, symbol Device:R_US
Connections:
- net 4IN1_EN renamed G1B5
- net G1B5: now also R14.1
- net 4IN1_LED renamed EXTMOD_LED
- net ELRS_BOOT renamed INTMOD_BOOT
- net ELRS_EN renamed INTMOD_EN
- net ELRS_LED renamed INTMOD_LED
- net PPM_I renamed EXTMOD_TX
- net PPM_O renamed EXTMOD_RX
- removed net PPM_RX_5V: J3.33 (Pin_33), J3.34 (Pin_34), J3.35 (Pin_35), J3.36 (Pin_36)
- net PPM_RX_EN renamed EXTMOD_EN
- net PPM_RX_LED renamed INT_PROTO_LED
- net INT_PROTO_LED: now also R14.2
Changed lines of the file:
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@@
 	)
 	(junction
-		(at 265.43 35.56)
-		(diameter 0)
-		(color 0 0 0 0)
-	)
-	(junction
 		(at 185.42 72.39)
 		(diameter 0)
@@
 	)
 	(junction
-		(at 265.43 33.02)
-		(diameter 0)
-		(color 0 0 0 0)
-	)
-	(junction
 		(at 24.13 54.61)
 		(diameter 0)
@@
 	(wire
 		(pts
-			(xy 265.43 30.48) (xy 265.43 33.02)
-		)
-		(stroke
-			(width 0)
-			(type default)
-		)
-	)
-	(wire
-		(pts
 			(xy 190.5 115.57) (xy 205.74 115.57)
 		)
@@
 	(wire
 		(pts
-			(xy 95.25 138.43) (xy 106.68 138.43)
+			(xy 95.25 138.43) (xy 120.65 138.43)
 		)
 		(stroke
@@
 	(wire
 		(pts
-			(xy 265.43 33.02) (xy 265.43 35.56)
-		)
-		(stroke
-			(width 0)
-			(type default)
-		)
-	)
-	(wire
-		(pts
 			(xy 241.3 93.98) (xy 265.43 93.98)
 		)
@@
 	(wire
 		(pts
-			(xy 265.43 35.56) (xy 265.43 38.1)
-		)
-		(stroke
-			(width 0)
-			(type default)
-		)
-	)
-	(wire
-		(pts
 			(xy 66.04 80.01) (xy 60.96 80.01)
 		)
@@
 		)
 	)
-	(text_box "LEDs:\n	VBUS -> CHARGING\n	VBUS -> CHG_DONE\n	PWR_EN -> GND\n	4IN1_LED -> GND\n	ELST_LED -> GND\n	PPM_RX_LED -> GND\n"
+	(text_box "LEDs:\n	VBUS -> CHARGING\n	VBUS -> CHG_DONE\n	PWR_EN -> GND\n	INT_PROTO_LED -> GND\n	INTMOD_LED -> GND\n	EXTMOD_LED -> GND\n"
 		(exclude_from_sim no)
 		(at 213.36 106.68 0)
@@
 	)
 	(global_label "PWR_SW_ON"
-		(shape input)
+		(shape bidirectional)
 		(at 265.43 43.18 180)
 		(fields_autoplaced yes)
@@
 		)
 		(property "Intersheetrefs" "${INTERSHEET_REFS}"
-			(at 251.1963 43.18 0)
+			(at 250.085 43.18 0)
 			(effects
 				(font
@@
 		)
 	)
-	(global_label "PPM_RX_LED"
+	(global_label "INT_PROTO_LED"
 		(shape input)
 		(at 190.5 110.49 180)
@@
 		)
 		(property "Intersheetrefs" "${INTERSHEET_REFS}"
-			(at 175.6616 110.49 0)
+			(at 173.061 110.49 0)
 			(effects
 				(font
@@
 		)
 	)
-	(global_label "VBUS"
-		(shape input)
-		(at 256.54 116.84 180)
+	(global_label "INT_PROTO_LED"
+		(shape output)
+		(at 128.27 138.43 0)
 		(fields_autoplaced yes)
 		(effects
@@
 				(size 1.27 1.27)
 			)
-			(justify right)
+			(justify left)
 		)
 		(property "Intersheetrefs" "${INTERSHEET_REFS}"
-			(at 248.6562 116.84 0)
+			(at 145.709 138.43 0)
 			(effects
 				(font
 					(size 1.27 1.27)
 				)
-				(justify right)
+				(justify left)
 				(hide yes)
 			)
 		)
 	)
-	(global_label "5V_PWR_EN"
+	(global_label "VBUS"
 		(shape input)
-		(at 106.68 130.81 0)
+		(at 256.54 116.84 180)
 		(fields_autoplaced yes)
 		(effects
@@
 				(size 1.27 1.27)
 			)
-			(justify left)
+			(justify right)
 		)
 		(property "Intersheetrefs" "${INTERSHEET_REFS}"
-			(at 120.3694 130.81 0)
+			(at 248.6562 116.84 0)
 			(effects
 				(font
 					(size 1.27 1.27)
 				)
-				(justify left)
+				(justify right)
 				(hide yes)
 			)
 		)
 	)
-	(global_label "4IN1_EN"
-		(shape input)
-		(at 106.68 138.43 0)
+	(global_label "5V_PWR_EN"
+		(shape output)
+		(at 106.68 130.81 0)
 		(fields_autoplaced yes)
 		(effects
@@
 		)
 		(property "Intersheetrefs" "${INTERSHEET_REFS}"
-			(at 117.4666 138.43 0)
+			(at 120.3694 130.81 0)
 			(effects
 				(font
@@
 		)
 	)
-	(global_label "PPM_O"
+	(global_label "EXTMOD_RX"
 		(shape input)
 		(at 257.81 91.44 180)
@@
 		)
 		(property "Intersheetrefs" "${INTERSHEET_REFS}"
-			(at 248.5353 91.44 0)
+			(at 243.9997 91.44 0)
 			(effects
 				(font
@@
 		)
 	)
-	(global_label "PPM_I"
-		(shape input)
+	(global_label "EXTMOD_TX"
+		(shape output)
 		(at 257.81 88.9 180)
 		(fields_autoplaced yes)
@@
 		)
 		(property "Intersheetrefs" "${INTERSHEET_REFS}"
-			(at 249.261 88.9 0)
+			(at 244.3021 88.9 0)
 			(effects
 				(font
@@
 		)
 	)
-	(global_label "ELRS_BOOT"
-		(shape input)
+	(global_label "INTMOD_BOOT"
+		(shape output)
 		(at 106.68 135.89 0)
 		(fields_autoplaced yes)
@@
 		)
 		(property "Intersheetrefs" "${INTERSHEET_REFS}"
-			(at 120.188 135.89 0)
+			(at 122.4862 135.89 0)
 			(effects
 				(font
@@
 	)
 	(global_label "ESP32_BOOT"
-		(shape input)
+		(shape output)
 		(at 262.89 96.52 180)
 		(fields_autoplaced yes)
@@
 		)
 	)
-	(global_label "4IN1_LED"
+	(global_label "EXTMOD_LED"
 		(shape input)
 		(at 190.5 100.33 180)
@@
 		)
 		(property "Intersheetrefs" "${INTERSHEET_REFS}"
-			(at 178.7458 100.33 0)
+			(at 175.7221 100.33 0)
 			(effects
 				(font
@@
 		)
 	)
-	(global_label "ELRS_LED"
+	(global_label "INTMOD_LED"
 		(shape input)
 		(at 190.5 97.79 180)
@@
 		)
 		(property "Intersheetrefs" "${INTERSHEET_REFS}"
-			(at 178.4435 97.79 0)
+			(at 176.1453 97.79 0)
 			(effects
 				(font
@@
 	)
 	(global_label "~{PWR_SW_DET}"
-		(shape input)
+		(shape bidirectional)
 		(at 265.43 40.64 180)
 		(fields_autoplaced yes)
@@
 		)
 		(property "Intersheetrefs" "${INTERSHEET_REFS}"
-			(at 250.4707 40.64 0)
-			(effects
-				(font
-					(size 1.27 1.27)
-				)
-				(justify right)
-				(hide yes)
-			)
-		)
-	)
-	(global_label "PPM_RX_5V"
-		(shape input)
-		(at 265.43 30.48 180)
-		(fields_autoplaced yes)
-		(effects
-			(font
-				(size 1.27 1.27)
-			)
-			(justify right)
-		)
-		(property "Intersheetrefs" "${INTERSHEET_REFS}"
-			(at 251.7406 30.48 0)
+			(at 249.3594 40.64 0)
 			(effects
 				(font
@@
 	)
 	(global_label "SDA"
-		(shape input)
+		(shape bidirectional)
 		(at 54.61 39.37 180)
 		(fields_autoplaced yes)
@@
 		)
 		(property "Intersheetrefs" "${INTERSHEET_REFS}"
-			(at 48.0567 39.37 0)
+			(at 46.9454 39.37 0)
 			(effects
 				(font
@@
 		)
 	)
-	(global_label "PPM_RX_EN"
-		(shape input)
+	(global_label "EXTMOD_EN"
+		(shape output)
 		(at 106.68 143.51 0)
 		(fields_autoplaced yes)
@@
 		)
 		(property "Intersheetrefs" "${INTERSHEET_REFS}"
-			(at 120.5508 143.51 0)
+			(at 120.4903 143.51 0)
 			(effects
 				(font
@@
 	)
 	(global_label "SDA"
-		(shape input)
+		(shape bidirectional)
 		(at 49.53 125.73 180)
 		(fields_autoplaced yes)
@@
 		)
 		(property "Intersheetrefs" "${INTERSHEET_REFS}"
-			(at 42.9767 125.73 0)
+			(at 41.8654 125.73 0)
 			(effects
 				(font
@@
 	)
 	(global_label "PWR_EN"
-		(shape input)
+		(shape output)
 		(at 106.68 140.97 0)
 		(fields_autoplaced yes)
@@
 	)
 	(global_label "PWR_SW_ON"
-		(shape input)
+		(shape output)
 		(at 205.74 143.51 0)
 		(fields_autoplaced yes)
@@
 	)
 	(global_label "RXD0"
-		(shape input)
+		(shape output)
 		(at 260.35 99.06 180)
 		(fields_autoplaced yes)
@@
 		)
 	)
-	(global_label "ELRS_EN"
-		(shape input)
+	(global_label "INTMOD_EN"
+		(shape output)
 		(at 106.68 133.35 0)
 		(fields_autoplaced yes)
@@
 		)
 		(property "Intersheetrefs" "${INTERSHEET_REFS}"
-			(at 117.7689 133.35 0)
+			(at 120.0671 133.35 0)
 			(effects
 				(font
@@
 	)
 	(global_label "SDA"
-		(shape input)
+		(shape bidirectional)
 		(at 190.5 105.41 180)
 		(fields_autoplaced yes)
@@
 		)
 		(property "Intersheetrefs" "${INTERSHEET_REFS}"
-			(at 183.9467 105.41 0)
+			(at 182.8354 105.41 0)
 			(effects
 				(font
@@
 	)
 	(global_label "~{PWR_SW_DET}"
-		(shape input)
+		(shape output)
 		(at 251.46 144.78 0)
 		(fields_autoplaced yes)
@@
 					(unit 1)
 				)
+			)
+		)
+	)
+	(symbol
+		(lib_id "Device:R_US")
+		(at 124.46 138.43 90)
+		(unit 1)
+		(exclude_from_sim no)
+		(in_bom yes)
+		(on_board yes)
+		(dnp no)
+		(property "Reference" "R14"
+			(at 124.46 140.97 90)
+			(effects
+				(font
+					(size 1.27 1.27)
+				)
+			)
+		)
+		(property "Value" "1K"
+			(at 124.46 143.002 90)
+			(effects
+				(font
+					(size 1.27 1.27)
+				)
+			)
+		)
+		(property "Footprint" "Resistor_SMD:R_0603_1608Metric_Pad0.98x0.95mm_HandSolder"
+			(at 124.714 137.414 90)
+			(effects
+				(font
+					(size 1.27 1.27)
+				)
+				(hide yes)
+			)
+		)
+		(property "Datasheet" "~"
+			(at 124.46 138.43 0)
+			(effects
+				(font
+					(size 1.27 1.27)
+				)
+				(hide yes)
+			)
+		)
+		(property "Description" "Resistor, US symbol"
+			(at 124.46 138.43 0)
+			(effects
+				(font
+					(size 1.27 1.27)
+				)
+				(hide yes)
+			)
+		)
+		(pin "1"
+		)
+		(pin "2"
+		)
+		(instances
+			(project "Muffin-Core"
+				(path "/f9f54452-72bc-42e0-a85c-2b2c5cedd536/b1aced65-cda0-4d30-b2f4-6d0180c9f383"
+					(reference "R14")
+					(unit 1)
+				)
