File: Muffin-Core/Muffin-Core.kicad_pcb (KiCad board)
At the start: 4 copper layers, 89 x 60 mm, 88 parts, among them J1 LCD, J10 Micro_SD_Card, J12 LIPO, J14 TouchPanel, J2 BUTTONS_AND_LEDS, J3 PWR_USB_PPM, J4 Gimbal, J5 4IN1, J6 ELRS, J7 Speaker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

Commit message: Fix issues found
Parts:
- removed C16: 1uF, Capacitor_SMD:C_0603_1608Metric_Pad1.08x0.95mm_HandSolder
- removed C23: 0.1uF, Capacitor_SMD:C_0603_1608Metric_Pad1.08x0.95mm_HandSolder
- removed R17: 1K, Resistor_SMD:R_0603_1608Metric_Pad0.98x0.95mm_HandSolder
- removed R20: 100K, Resistor_SMD:R_0603_1608Metric_Pad0.98x0.95mm_HandSolder
- removed R28: 0, Resistor_SMD:R_0603_1608Metric_Pad0.98x0.95mm_HandSolder
- removed U9: SiP32431DR3, Package_TO_SOT_SMD:SOT-363_SC-70-6
- added R14: 1K, Resistor_SMD:R_0603_1608Metric_Pad0.98x0.95mm_HandSolder, F.Cu at (102.4, 67.2)
- J4: footprint Connector_Molex:Molex_PicoBlade_53398-0471_1x04-1MP_P1.25mm_Vertical -> Connector_JST:JST_ZH_B4B-ZR-SM4-TF_1x04-1MP_P1.50mm_Vertical
- J5: value 4IN1 -> ELRS; footprint Connector_Molex:Molex_PicoBlade_53398-0471_1x04-1MP_P1.25mm_Vertical -> Connector_Molex:Molex_PicoBlade_53398-0571_1x05-1MP_P1.25mm_Vertical
- R12, R13: value 100K -> 1K
- moved C17 58.2 mm to (143.9, 58.3), turned to 90 degrees
- moved C24 56.5 mm to (147.4, 62.2)
- moved J6 55.8 mm to (151.8, 65.2)
- moved U10 54.9 mm to (144.9, 61.8), turned to 180 degrees
- moved R23 53.9 mm to (146.4, 64.6), turned to 180 degrees
- moved C22 28.5 mm to (90.2, 67.0), turned to 90 degrees
- moved C25 26.2 mm to (93.7, 69.3)
- moved R24 26.2 mm to (93.7, 70.8)
- moved U11 26.2 mm to (89.6, 70.3)
- moved D2 17.2 mm to (161.0, 57.1)
- moved R29 17.2 mm to (153.0, 55.1)
- moved R5 17.2 mm to (164.6, 55.3)
- moved C12 17.2 mm to (157.2, 60.7)
- moved C7 17.2 mm to (164.2, 61.7)
- moved C9 17.2 mm to (157.2, 67.7)
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Connections:
- net /ESP32/GIMBAL_RX renamed GIMBAL_RX
- net /ESP32/GIMBAL_TX renamed GIMBAL_TX
- net ELRS_5V renamed INTMOD_5V
- net ELRS_BOOT renamed INTMOD_BOOT
- net ELRS_EN renamed INTMOD_EN
- net ELRS_LED renamed INTMOD_LED
- net PPM_RX_EN renamed EXTMOD_EN
- C25 pad 2: PPM_RX_5V -> EXTMOD_5V
- J1 pad 12: /ESP32/LCD_RD -> +3.3V
- J14 pad 5: Net-(J14-Pin_5) -> ~{RESET}
- J2 pad 32: 4IN1_LED -> EXTMOD_LED
- J2 pad 36: PPM_RX_LED -> INT_PROTO_LED
- J3 pad 12: PPM_O -> EXTMOD_RX
- J3 pad 13: PPM_I -> EXTMOD_TX
- J3 pad 33: PPM_RX_5V -> unconnected-(J3-Pin_33-Pad33)
- J3 pad 34: PPM_RX_5V -> unconnected-(J3-Pin_34-Pad34)
- J3 pad 35: PPM_RX_5V -> unconnected-(J3-Pin_35-Pad35)
- J3 pad 36: PPM_RX_5V -> unconnected-(J3-Pin_36-Pad36)
- J5 pad 1: INTMOD_TX -> unconnected-(J5-Pin_1-Pad1)
- J5 pad 2: INTMOD_RX -> EXTMOD_TX
- J5 pad 3: GND -> EXTMOD_RX
- J5 pad 4: 4IN1_5V -> GND
- R24 pad 1: PPM_RX_5V -> EXTMOD_5V
- R24 pad 2: PPM_RX_LED -> EXTMOD_LED
- U1 pad 12: PPM_O -> EXTMOD_RX
- U1 pad 8: PPM_I -> EXTMOD_TX
- U11 pad 1: PPM_RX_5V -> EXTMOD_5V
- U3 pad 2: 4IN1_EN -> /GPIO_ext/G1B5
Routing:
- net EXTMOD_TX: track 0.00 -> 90.1 mm, vias 0 -> 2
- net EXTMOD_RX: track 0.00 -> 85.8 mm, vias 0 -> 2
- net INTMOD_TX: track 104.9 -> 25.6 mm, vias 3 -> 2
- net INTMOD_RX: track 106.2 -> 27.4 mm, vias 3 -> 2
- net 4IN1_LED: track 65.8 -> 0.00 mm
- net PPM_I: track 64.4 -> 0.00 mm, vias 2 -> 0
- net PPM_O: track 62.4 -> 0.00 mm, vias 2 -> 0
- net PPM_RX_LED: track 57.1 -> 0.00 mm, vias 2 -> 0
- net INTMOD_BOOT: track 12.6 -> 68.3 mm, vias 0 -> 2
- net EXTMOD_LED: track 0.00 -> 49.3 mm, vias 0 -> 2
- net ~{RESET}: track 125.9 -> 171.1 mm, vias 5 -> 9
- net INTMOD_EN: track 16.8 -> 59.6 mm, vias 0 -> 2
- net PWR_EN: track 111.8 -> 75.1 mm
- net INT_PROTO_LED: track 0.00 -> 35.2 mm, vias 0 -> 2
- net 4IN1_EN: track 22.9 -> 0.00 mm
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- removed copper zone on F.Cu, net 4IN1_5V
- removed copper zone on F.Cu, net INTMOD_5V
- removed copper zone on F.Cu, net PPM_RX_5V
Other:
- outline, holes or cut-outs redrawn
- board text added: "PCB Muffin v1.1"
- board text removed: "PCB Muffin v1.0"
