File: Muffin-Core/esp32.kicad_sch (KiCad schematic)
At the start: 26 parts, among them J1 LCD, J10 Micro_SD_Card, J14 TouchPanel, J4 Gimbal, J5 4IN1, J6 ELRS, J9 USB_C, Q1 AO3400A, U1 ESP32-S3-WROOM-1U, U6 DS3231MZ

Commit message: Fix issues found
Parts:
- removed J5: 4IN1, Connector_Molex:Molex_PicoBlade_53398-0471_1x04-1MP_P1.25mm_Vertical, symbol Connector_Generic:Conn_01x04
- removed R20: 100K, Resistor_SMD:R_0603_1608Metric_Pad0.98x0.95mm_HandSolder, symbol Device:R_US
- removed R28: 0, Resistor_SMD:R_0603_1608Metric_Pad0.98x0.95mm_HandSolder, symbol Device:R_US
- added J5: ELRS, Connector_Molex:Molex_PicoBlade_53398-0571_1x05-1MP_P1.25mm_Vertical, symbol Connector_Generic:Conn_01x05
- J4: footprint Connector_Molex:Molex_PicoBlade_53398-0471_1x04-1MP_P1.25mm_Vertical -> Connector_JST:JST_ZH_B4B-ZR-SM4-TF_1x04-1MP_P1.50mm_Vertical
Connections:
- net LCD_RD is gone; now on net +3.3V: J1.12 (Pin_12)
- net GND: now also J5.4 (Pin_4)
- net ~{RESET}: now also J14.5 (Pin_5)
- net ELRS_5V renamed INTMOD_5V
- net ELRS_BOOT renamed INTMOD_BOOT
- net PPM_I renamed EXTMOD_TX
- net EXTMOD_TX: now also J5.2 (Pin_2)
- net PPM_O renamed EXTMOD_RX
- net EXTMOD_RX: now also J5.3 (Pin_3)
- new net EXTMOD_5V: J5.5 (Pin_5)
