File: Muffin-Core/power.kicad_sch (KiCad schematic)
At the start: 43 parts, among them J12 LIPO, U10 SiP32431DR3, U11 SiP32431DR3, U4 TPS62827DMQR, U5 TPS61023DRLR, U7 MCP73871, U9 SiP32431DR3

Commit message: Fix issues found
Parts:
- removed C16: 1uF, Capacitor_SMD:C_0603_1608Metric_Pad1.08x0.95mm_HandSolder, symbol Adafruit PowerBoost 1000C Rev B-eagle-import:CAP_CERAMIC0805-NOOUTLINE
- removed C23: 0.1uF, Capacitor_SMD:C_0603_1608Metric_Pad1.08x0.95mm_HandSolder, symbol Adafruit PowerBoost 1000C Rev B-eagle-import:CAP_CERAMIC0805-NOOUTLINE
- removed R17: 1K, Resistor_SMD:R_0603_1608Metric_Pad0.98x0.95mm_HandSolder, symbol Device:R_US
- removed U9: SiP32431DR3, Package_TO_SOT_SMD:SOT-363_SC-70-6, symbol Power_Management:SiP32431DR3
- R12, R13: value 100K -> 1K
Connections:
- net ELRS_5V renamed INTMOD_5V
- net ELRS_EN renamed INTMOD_EN
- net ELRS_LED renamed INTMOD_LED
- net PPM_RX_5V renamed EXTMOD_5V
- net PPM_RX_EN renamed EXTMOD_EN
- net PPM_RX_LED renamed EXTMOD_LED
Other:
- moved on the sheet: C17, C24, R23, U10
