File: Muffin/Muffin.kicad_pcb (KiCad board)
At the start: 4 copper layers, 145.5 x 64 mm, 138 parts, among them J1 USB_C, J10 I2C_STEMMA, J11 TRAINER, J12 Gimbal, J13 USB_C, J15 EXTMOD, J17 Micro_SD_Card, J18 INTMOD, J19 TouchPanel, J2 SWB, J20 LCD, J21 LIPO, J24 Speaker, J3 SWA, J4 SWC, J5 SWD, J6 VRA, J7 VRB, J8 TRIMS, J9 LEDs, Q1 MBT3904DW1, Q2 AO3400A, SW1 TRRIM_RUD_LEFT, SW10 SW_Slide_DPDT, SW2 TRIM_RUD_RIGHT, SW3 TRIM_AIL_LEFT, SW4 TRIM_AIL_RIGHT, SW5 KEY_ENTER, SW6 KEY_EXIT, SW7 KEY_UP, SW8 KEY_DOWN, SW9 KEY_MENU, U1 CP2102N-Axx-xQFN24, U10 MCP73871, U11 MCP23017_ML, U12 MCP23017_ML, U13 MAX98357A, U2 ADS1015IDGS, U3 ADS1015IDGS, U4 ESP32-S3-WROOM-1U, U5 DS3231MZ, U6 SiP32431DR3, U7 TPS62827DMQR, U8 TPS61023DRLR, U9 SiP32431DR3

Commit message: PCB 2.1
Fixed a reversed ZH-socket on the board for Gimbal
Connections:
- J12 pad 1: GND -> +3.3V
- J12 pad 2: /ESP32 Core/GIMBAL_TX -> /ESP32 Core/GIMBAL_RX
- J12 pad 3: /ESP32 Core/GIMBAL_RX -> /ESP32 Core/GIMBAL_TX
- J12 pad 4: +3.3V -> GND
Routing:
- net /ESP32 Core/GIMBAL_RX: track 22.2 -> 25.6 mm
- net /ESP32 Core/GIMBAL_TX: track 22.3 -> 21.7 mm
Other:
- board text added: "PCB Muffin v2.1"
- board text removed: "PCB Muffin v2.0"
Changed lines of the file:
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@@
 			(layers "F.Cu" "F.Paste" "F.Mask")
 			(roundrect_rratio 0.25)
-			(net 2 "GND")
+			(net 1 "+3.3V")
 			(pinfunction "Pin_1")
 			(pintype "passive")
@@
 			(layers "F.Cu" "F.Paste" "F.Mask")
 			(roundrect_rratio 0.25)
-			(net 88 "/ESP32 Core/GIMBAL_TX")
+			(net 89 "/ESP32 Core/GIMBAL_RX")
 			(pinfunction "Pin_2")
 			(pintype "passive")
@@
 			(layers "F.Cu" "F.Paste" "F.Mask")
 			(roundrect_rratio 0.25)
-			(net 89 "/ESP32 Core/GIMBAL_RX")
+			(net 88 "/ESP32 Core/GIMBAL_TX")
 			(pinfunction "Pin_3")
 			(pintype "passive")
@@
 			(layers "F.Cu" "F.Paste" "F.Mask")
 			(roundrect_rratio 0.25)
-			(net 1 "+3.3V")
+			(net 2 "GND")
 			(pinfunction "Pin_4")
 			(pintype "passive")
@@
 			(roundrect_rratio 0.166667)
 		)
-		(model "${KICAD8_3DMODEL_DIR}/Connector_JST.3dshapes/JST_ZH_B4B-ZR-SM4-TF_1x04-1MP_P1.50mm_Vertical.wrl"
+		(model "C:/Users/ollyl/OneDrive/RC_plane/edgetx/PCB/my_footprints.pretty/ZH_SMT_VERTICAL_4pin.step"
 			(offset
-				(xyz 0 0 0)
+				(xyz 0 -0.5 0)
 			)
 			(scale
@@
 			(roundrect_rratio 0.138889)
 		)
-		(model "${KICAD8_3DMODEL_DIR}/Connector_JST.3dshapes/JST_ZE_BM03B-ZESS-TBT_1x03-1MP_P1.50mm_Vertical.wrl"
+		(model "C:/Users/ollyl/OneDrive/RC_plane/edgetx/PCB/my_footprints.pretty/ZH_SMT_VERTICAL_6pin.step"
 			(offset
-				(xyz 0 0 0)
+				(xyz 2.3 -3.5 0)
 			)
 			(scale
@@
 			(thermal_bridge_angle 45)
 		)
+		(model "C:/Users/ollyl/OneDrive/RC_plane/edgetx/PCB/my_footprints.pretty/FPC_6PIN_BOTTOM v5.step"
+			(offset
+				(xyz 0 0 0)
+			)
+			(scale
+				(xyz 1 1 1)
+			)
+			(rotate
+				(xyz 0 0 0)
+			)
+		)
 	)
 	(footprint "my_footprints:MicroSD"
@@
 			(roundrect_rratio 0.138889)
 		)
-		(model "${KICAD8_3DMODEL_DIR}/Connector_JST.3dshapes/JST_ZE_BM03B-ZESS-TBT_1x03-1MP_P1.50mm_Vertical.wrl"
+		(model "C:/Users/ollyl/OneDrive/RC_plane/edgetx/PCB/my_footprints.pretty/ZH_SMT_VERTICAL_6pin.step"
 			(offset
-				(xyz 0 0 0)
+				(xyz 2.3 -3.5 0)
 			)
 			(scale
@@
 			(roundrect_rratio 0.208333)
 		)
-		(model "${KICAD8_3DMODEL_DIR}/Connector_JST.3dshapes/JST_SH_BM04B-SRSS-TB_1x04-1MP_P1.00mm_Vertical.wrl"
+		(model "C:/Users/ollyl/OneDrive/RC_plane/edgetx/PCB/my_footprints.pretty/SH-SMT_4pin.step"
 			(offset
-				(xyz 0 0 0)
+				(xyz 0 0.5 0)
 			)
 			(scale
@@
 		(layer "Edge.Cuts")
 	)
-	(gr_text "PCB Muffin v2.0"
+	(gr_text "PCB Muffin v2.1"
 		(at 97.6 104.8 0)
 		(layer "F.SilkS")
@@
 	)
 	(via
-		(at 126.6 54.4)
+		(at 100.85 89.799998)
 		(size 0.6)
 		(drill 0.3)
@@
 	)
 	(via
-		(at 100.85 89.799998)
+		(at 122.1 54.4)
 		(size 0.6)
 		(drill 0.3)
@@
 	)
 	(via
-		(at 122.1 54.4)
+		(at 67.2 61.6)
 		(size 0.6)
 		(drill 0.3)
 		(layers "F.Cu" "B.Cu")
+		(free yes)
 		(net 2)
 	)
 	(via
-		(at 67.2 61.6)
+		(at 126.6 54.4)
 		(size 0.6)
 		(drill 0.3)
 		(layers "F.Cu" "B.Cu")
-		(free yes)
 		(net 2)
 	)
@@
 	)
 	(via
-		(at 123.6 54.4)
+		(at 125.1 54.4)
 		(size 0.6)
 		(drill 0.3)
@@
 	)
 	(segment
-		(start 129.3 74.345606)
-		(end 129.3 60.1)
+		(start 129.3 58.6)
+		(end 125.1 54.4)
 		(width 0.2)
 		(layer "B.Cu")
@@
 	)
 	(segment
-		(start 129.3 60.1)
-		(end 123.6 54.4)
+		(start 129.3 74.345606)
+		(end 129.3 58.6)
 		(width 0.2)
 		(layer "B.Cu")
@@
 	)
 	(via
-		(at 125.1 54.4)
+		(at 123.6 54.4)
 		(size 0.6)
 		(drill 0.3)
@@
 	)
 	(segment
-		(start 130.57 59.87)
-		(end 125.1 54.4)
+		(start 130.57 74.345606)
+		(end 130.57 57.521471)
 		(width 0.2)
 		(layer "B.Cu")
@@
 	)
 	(segment
-		(start 130.57 74.345606)
-		(end 130.57 59.87)
+		(start 130.57 57.521471)
+		(end 126.848529 53.8)
+		(width 0.2)
+		(layer "B.Cu")
+		(net 89)
+	)
+	(segment
+		(start 124.2 53.8)
+		(end 123.6 54.4)
+		(width 0.2)
+		(layer "B.Cu")
+		(net 89)
+	)
+	(segment
+		(start 126.848529 53.8)
+		(end 124.2 53.8)
 		(width 0.2)
 		(layer "B.Cu")
